File: wav_man_dev_board_v1.kicad_sch (KiCad schematic)
At the start: 27 parts, among them J1 Micro_SD_Card, J4 BATTERY, P1 USB_C_Plug_USB2.0, SW16 PWR_SW, U2 AZ1117-3.3, U3 ATSAMD21G18A-A

Commit message: updated schematic with v1 changes: fixed DAC power, added debug port, fixed mute and hold functionality
Parts:
- added J2: DEBUG, Connector_PinSocket_2.54mm:PinSocket_1x06_P2.54mm_Vertical, symbol Connector:Conn_01x06_Socket
- renumbered 32MHz1 to 32.768kHz
Connections:
- net 3.3V: now also J2.2 (Pin_2)
- net DISP_SEG_A: now also J2.6 (Pin_6)
- net DISP_SEG_B: now also J2.5 (Pin_5)
- net DISP_SEG_DOT: now also J2.4 (Pin_4)
- net DISP_SEG_G: now also J2.3 (Pin_3)
- net GND: now also J2.1 (Pin_1)
- net PCM_MUTE: now reaches U3.10 (PA05)
- net HOLD: now reaches U3.11 (PA06)
Other:
- note added: "Optional Oscillator"
- note removed: "HOLD is not wired to anything"
- note removed: "We probably don't need all this shit"
- note removed: "XIN/XOUT on PA00 and PA01 uses a 32.768kHz oscillator"
- company: (none) -> MCRAE/JONES
- title: (none) -> WAVMAN
- moved on the sheet: TP4

Commit message: usb fixed, rerouted some traces
Parts:
- removed TP1, TP4, TP5: TP_GND, TestPoint:TestPoint_Pad_2.0x2.0mm, symbol Connector:TestPoint
- removed TP2: TP_3V3, TestPoint:TestPoint_Pad_2.0x2.0mm, symbol Connector:TestPoint
- removed TP3: TP_CLK, TestPoint:TestPoint_Pad_2.0x2.0mm, symbol Connector:TestPoint
- C13, C19, C20, C21, C22, C23, C24, C25, C26: footprint Capacitor_SMD:C_1206_3216Metric_Pad1.33x1.80mm_HandSolder -> Capacitor_SMD:C_0805_2012Metric_Pad1.18x1.45mm_HandSolder
- P1: symbol Connector:USB_C_Plug_USB2.0 -> Connector:USB_C_Receptacle_USB2.0_16P
- R37: footprint Resistor_SMD:R_1206_3216Metric_Pad1.30x1.75mm_HandSolder -> Resistor_SMD:R_0805_2012Metric_Pad1.20x1.40mm_HandSolder
- renumbered 32.768kHz to 32.768kHz1
Connections:
- net USB_DM: now also P1.B7 (D-)
- net USB_DP: now also P1.B6 (D+)

Commit message: minor fixes to audio amp, updated readme
Connections:
- no-connect marks 0 -> 3
Other:
- note added: "Power is not supplied via USB"
Changed lines of the file:
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@@
+		)
+	)
+	(text "Power is not supplied via USB"
+		(exclude_from_sim no)
+		(at 265.684 97.79 0)
+		(effects
+			(font
+				(size 1.27 1.27)
+			)
 		)
 	)
@@
 		(color 0 0 0 0)
 	)
+	(no_connect
+		(at 255.27 109.22)
+	)
+	(no_connect
+		(at 255.27 104.14)
+	)
+	(no_connect
+		(at 255.27 111.76)
+	)
 	(wire
